File: Peripherals.kicad_sch (KiCad schematic)
At the start: 26 parts, among them J2 Conn_01x02, M1 Vibrator DC Motor, U1 MAX30102, U10 DRV2603RUNR, U2 BMI270, U3 OPT3004DNPR, U4 LPS22DF, U5 W25Q32JVSS

Commit message: Layout V1
Connections:
- net MOTOR+: now reaches J2.1 (Pin_1), U10.9 (OUT+)
- net MOTOR-: now reaches J2.2 (Pin_2), U10.6 (OUT-)
Other:
- moved on the sheet: J2
Changed lines of the file:
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@@
 	(wire
 		(pts
-			(xy 226.06 107.95) (xy 229.87 107.95)
+			(xy 226.06 107.95) (xy 233.68 107.95)
 		)
 		(stroke
@@
 	(wire
 		(pts
-			(xy 226.06 105.41) (xy 229.87 105.41)
+			(xy 226.06 105.41) (xy 233.68 105.41)
 		)
 		(stroke
@@
 			(width 0)
 			(type default)
+		)
+	)
+	(label "MOTOR+"
+		(at 226.06 105.41 0)
+		(effects
+			(font
+				(size 1.27 1.27)
+			)
+			(justify left bottom)
+		)
+	)
+	(label "MOTOR-"
+		(at 226.06 107.95 0)
+		(effects
+			(font
+				(size 1.27 1.27)
+			)
+			(justify left bottom)
 		)
 	)
@@
 	(symbol
 		(lib_id "Connector_Generic:Conn_01x02")
-		(at 234.95 105.41 0)
+		(at 238.76 105.41 0)
 		(unit 1)
 		(body_style 1)
@@
 		(fields_autoplaced yes)
 		(property "Reference" "J2"
-			(at 236.982 105.4678 0)
+			(at 240.792 105.4678 0)
 			(show_name no)
 			(do_not_autoplace no)
@@
 		)
 		(property "Value" "Conn_01x02"
-			(at 236.982 107.8921 0)
+			(at 240.792 107.8921 0)
 			(show_name no)
 			(do_not_autoplace no)
@@
 		)
 		(property "Footprint" "PAD_CONNECTOR:1x02_1x1mm"
-			(at 234.95 105.41 0)
+			(at 238.76 105.41 0)
 			(hide yes)
 			(show_name no)
@@
 		)
 		(property "Datasheet" ""
-			(at 234.95 105.41 0)
+			(at 238.76 105.41 0)
 			(hide yes)
 			(show_name no)
@@
 		)
 		(property "Description" "Generic connector, single row, 01x02, script generated (kicad-library-utils/schlib/autogen/connector/)"
-			(at 234.95 105.41 0)
-			(hide yes)
-			(show_name no)
+			(at 238.76 105.41 0)
+			(hide yes)
+			(show_name no)
